File: Analog-Video-Comb-Filter/Analog-Video-Comb-Filter.kicad_sch (KiCad schematic)
At the start: 80 parts, among them J1 12VDC(+), J2 SVHS, J3 CV-OUT, J4 CV-IN, Q1 BC548, U1 L7805, U2 AD8044, U3 SAA4960/61, U4 MC44144, U5 74HC04, U6 LM1881, U7 SAA4963, Y1 See table

Commit message: Revision 3
- Settled on AD813 as the output amplifier, this should also fix #1 as AD8044 is no longer used;
- Added output gain adjustment.
Parts:
- removed JP1: ALT, Jumper:SolderJumper-2_P1.3mm_Open_RoundedPad1.0x1.5mm, symbol Jumper:SolderJumper_2_Open
- removed U2: AD8044, Package_DIP:DIP-14_W7.62mm_Socket, symbol Device:Opamp_Quad
- added RV1, RV2, RV3: 1k, Potentiometer_THT:Potentiometer_Piher_PT-10-H01_Horizontal, symbol Device:R_Potentiometer
- added U2: AD813, Package_DIP:DIP-14_W7.62mm_Socket, symbol Amplifier_Video:AD813
- R5, R6, R7: value 1k -> 470R
- renumbered JP2 to JP1, JP3 to JP2, JP4 to JP3, JP5 to JP4
Connections:
- net +12VA: now also U2.4 (V+)
- net CO: now also U2.5 (+)
- net CVO: now also U2.12 (+)
- net GND: now also U2.11 (V-)
- net YO: now also U2.10 (+)
- net at R4.2: now also RV3.1, RV3.2, U2.14; no longer R7.1
- net at R13.1, R7.2: now also U2.13 (-)
- net at R2.2: now also RV1.3, U2.7; no longer R5.1
- net at R5.2, R9.1: now also U2.6 (-)
- net at R3.2: now also RV2.1, RV2.2, U2.8; no longer R6.1
- net at R11.1, R6.2: now also U2.9 (-)
- new net: R7.1, RV3.3
- new net: R5.1, RV1.1, RV1.2
- new net: R6.1, RV2.3
- no-connect marks 18 -> 21
Other:
- moved on the sheet: J2, J3, R10, R11, R12, R2, R3, R4, R7, R8, R9, U5G
